File: PCB_screwSwitch/PCB_screwSwitch.kicad_sch (KiCad schematic)
At the start: 4 parts, among them J1 XT30PW-M, J2 Screw_Terminal_01x02

Commit message: Rev 3
Created rev A of custom PCB Switch
Parts:
- H2: footprint (none) -> parts_footprints:hole_bottom
Changed lines of the file:
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@@
 			)
 		)
-		(property "Footprint" ""
+		(property "Footprint" "parts_footprints:hole_bottom"
 			(at 118.11 81.28 0)
 			(effects
